File: pcb/sao_vapeorwear.kicad_pcb (KiCad board)
At the start: 2 copper layers, 48 x 46 mm, 26 parts, among them J1 USB_C_Receptacle_PowerOnly_6P, J2 Conn_01x02_MountingPin, J4 Conn_01x08_Pin, SW1 SW_SPDT, U1 MT3406, U2 any4054, U4 RY2201, X1 Simple_Addon_v2

Commit message: Better documentation
Parts:
- C1, C2, C3: value 22uF -> 10uF
- R1: value 220k -> 21k
- R11: value 5.1k -> 4.7k
- R14, R4: value 5.1k -> 560R
- R15: value 100R -> 560R
- R2: value 47k -> 4.7k
- R3: value 220k -> 4.7k
Other:
- board text added: "2x10uF"
- board text removed: "2x22uF"

Commit message: component values
Parts:
- C9: value 1uF -> 100nF
- R1: value 21k -> 22k
- R11: value 4.7k -> 2.2k
- R14, R4: value 560R -> 2.2k
- R15: value 560R -> 1k
Changed lines of the file:
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@@
 		)
 		(property "Value" "5.1k"
-			(at 0.1 -2.4 180)
+			(at -0.8 2.3 180)
 			(layer "F.Fab")
 			(effects
@@
 		)
 		(property "Value" "5.1k"
-			(at 0.1 2.4 180)
+			(at 1.1 -2.3 180)
 			(layer "F.Fab")
 			(effects
@@
 			)
 		)
-		(property "Value" "21k"
+		(property "Value" "22k"
 			(at -0.4 -1.5 0)
 			(layer "F.Fab")
@@
 			)
 		)
-		(property "Value" "560R"
+		(property "Value" "2.2k"
 			(at -3.4 0.1 0)
 			(layer "F.Fab")
@@
 			)
 		)
-		(property "Value" "560R"
+		(property "Value" "2.2k"
 			(at 3.4 0.1 0)
 			(layer "F.Fab")
@@
 			)
 		)
-		(property "Value" "560R"
+		(property "Value" "1k"
 			(at -0.5 -1.5 0)
 			(layer "F.Fab")
@@
 			)
 		)
-		(property "Value" "1uF"
-			(at -1.7 -0.2 180)
+		(property "Value" "100nF"
+			(at -0.6 -3.1 180)
 			(layer "F.Fab")
 			(effects
@@
 			)
 		)
-		(property "Value" "4.7k"
+		(property "Value" "2.2k"
 			(at 0 1.43 0)
 			(layer "F.Fab")
@@
 		)
 		(min_thickness 0.3)
-		(fill
+		(fill yes
 			(thermal_gap 0.3)
 			(thermal_bridge_width 0.8)
@@
 		)
 		(min_thickness 0.25)
-		(fill
+		(fill yes
 			(thermal_gap 0.5)
 			(thermal_bridge_width 0.5)
@@
 		)
 		(min_thickness 0.25)
-		(fill
+		(fill yes
 			(thermal_gap 0.5)
 			(thermal_bridge_width 0.5)
