File: pcb/sao_vapeorwear.kicad_sch (KiCad schematic)
At the start: 25 parts, among them J1 USB_C_Receptacle_PowerOnly_6P, J2 Conn_01x02_MountingPin, J4 Conn_01x08_Pin, SW1 SW_SPDT, U1 MT3406, U2 any4054, U4 RY2201, X1 Simple_Addon_v2

Commit message: Better documentation
Parts:
- C1, C2, C3: value 22uF -> 10uF
- R1: value 220k -> 21k
- R11: value 5.1k -> 4.7k
- R14, R4: value 5.1k -> 560R
- R15: value 100R -> 560R
- R2: value 47k -> 4.7k
- R3: value 220k -> 4.7k
Changed lines of the file:
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@@
 			)
 		)
-		(property "Value" "22uF"
+		(property "Value" "10uF"
 			(at 119.634 133.096 0)
 			(show_name no)
@@
 			)
 		)
-		(property "Value" "47k"
+		(property "Value" "4.7k"
 			(at 101.854 142.24 0)
 			(show_name no)
@@
 			)
 		)
-		(property "Value" "5.1k"
+		(property "Value" "560R"
 			(at 114.554 49.784 0)
 			(show_name no)
@@
 			)
 		)
-		(property "Value" "220k"
+		(property "Value" "21k"
 			(at 102.362 133.604 0)
 			(show_name no)
@@
 			)
 		)
-		(property "Value" "220k"
+		(property "Value" "4.7k"
 			(at 52.832 134.874 0)
 			(show_name no)
@@
 			)
 		)
-		(property "Value" "5.1k"
+		(property "Value" "560R"
 			(at 143.51 132.08 0)
 			(show_name no)
@@
 			)
 		)
-		(property "Value" "5.1k"
+		(property "Value" "4.7k"
 			(at 114.046 73.66 0)
 			(show_name no)
@@
 			)
 		)
-		(property "Value" "100R"
+		(property "Value" "560R"
 			(at 205.74 51.816 90)
 			(show_name no)
@@
 			)
 		)
-		(property "Value" "22uF"
+		(property "Value" "10uF"
 			(at 32.004 133.35 0)
 			(show_name no)
@@
 			)
 		)
-		(property "Value" "22uF"
+		(property "Value" "10uF"
 			(at 108.966 132.842 0)
 			(show_name no)

Commit message: component values
Parts:
- C9: value 1uF -> 100nF
- R1: value 21k -> 22k
- R11: value 4.7k -> 2.2k
- R14, R4: value 560R -> 2.2k
- R15: value 560R -> 1k
Other:
- note added: "Battery charging current is 1000/R11 Example: 2.0k -> 500mA (max allowed current) 2.2k -> 454mA (recommended) 4.7k -> 212mA (included in kit)"
- note added: "Vout = 0.6V * (1+(R1/R2)) Example: 0.6 * (1+(22000/4700)) = 3.41V The output is a bit hot, but for many SAOs that just means brighter LEDs!"
- note removed: "Vfb = 0.6V 0.6 / (47 / (47+220)) = 3.4V The output is a bit hot, but for many SAOs that just means brighter LEDs!"
Changed lines of the file:
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@@
 		)
 	)
-	(text "Vfb = 0.6V\n0.6 / (47 / (47+220)) = 3.4V\nThe output is a bit hot,\nbut for many SAOs that just means brighter LEDs!"
+	(text "Vout = 0.6V * (1+(R1/R2))\nExample:  0.6 * (1+(22000/4700)) = 3.41V\nThe output is a bit hot, but for many SAOs that just means brighter LEDs!"
 		(exclude_from_sim no)
-		(at 58.42 165.354 0)
+		(at 52.578 165.1 0)
+		(effects
+			(font
+				(size 1.27 1.27)
+			)
+			(justify left)
+		)
+	)
+	(text "Battery charging current is 1000/R11\nExample:\n2.0k -> 500mA (max allowed current)\n2.2k -> 454mA (recommended)\n4.7k -> 212mA (included in kit)\n"
+		(exclude_from_sim no)
+		(at 112.522 92.71 0)
 		(effects
 			(font
@@
 			)
 		)
-		(property "Value" "560R"
+		(property "Value" "2.2k"
 			(at 114.554 49.784 0)
 			(show_name no)
@@
 			)
 		)
-		(property "Value" "1uF"
+		(property "Value" "100nF"
 			(at 206.502 60.96 0)
 			(show_name no)
@@
 			)
 		)
-		(property "Value" "21k"
+		(property "Value" "22k"
 			(at 102.362 133.604 0)
 			(show_name no)
@@
 			)
 		)
-		(property "Value" "560R"
+		(property "Value" "2.2k"
 			(at 143.51 132.08 0)
 			(show_name no)
@@
 			)
 		)
-		(property "Value" "4.7k"
+		(property "Value" "2.2k"
 			(at 114.046 73.66 0)
 			(show_name no)
@@
 			)
 		)
-		(property "Value" "560R"
+		(property "Value" "1k"
 			(at 205.74 51.816 90)
 			(show_name no)
